Commit message: sync state

File: foxy_description/sensors/imu_generic.xacro (robot description, xacro)
@@ -13,5 +13,5 @@
       <xacro:insert_block name="origin" />
     </joint>
-    <xacro:if value="${system == 'gz'}">
+    <xacro:if value="${system == 'sim'}">
       <gazebo>
         <plugin filename="gz-sim-imu-system"

File: foxy_description/sensors/lidar_generic.xacro (robot description, xacro)
@@ -13,5 +13,5 @@
       <xacro:insert_block name="origin" />
     </joint>
-    <xacro:if value="${system == 'gz'}">
+    <xacro:if value="${system == 'sim'}">
       <gazebo reference="${name}_link">
         <sensor name="${name}_link" type='gpu_lidar'>"

File: foxy_description/sensors/rgb_camera_generic.xacro (robot description, xacro)
@@ -13,5 +13,5 @@
       <xacro:insert_block name="origin" />
     </joint>
-    <xacro:if value="${system == 'gz'}">
+    <xacro:if value="${system == 'sim'}">
       <gazebo reference="${name}_link">
         <plugin filename="gz-sim-imu-system"

File: foxy_description/urdf/base.xacro (robot description, xacro)
@@ -73,4 +73,5 @@
       <child link="base_footprint" />
       <origin xyz="0 0 ${-(wheel_radius+wheel_zoff)}" rpy="0 0 0" />
+      <dynamics friction="1.0"/>
     </joint>
     <xacro:wheel prefix="left_wheel" parent="${root_frame}" x_reflect="1" y_reflect="1" />

File: foxy_description/urdf/foxy.urdf.xacro (robot description, xacro)
@@ -8,5 +8,7 @@
   <!-- <xacro:property name="root_frame" default="${namespace}/base_link" /> -->
   <xacro:property name="root_frame" default="base_link" />
-  <xacro:property name="ros2_gz_before_renamed" value="${['humble', 'galatic', 'foxy']}"/>
+  <xacro:property name="ros2_gz_before_renamed" value="${['humble', 'jazzy', 'kilted']}"/>
+  <!-- HARLEY DEBUG: removing humble in my setup -->
+  <!-- <xacro:property name="ros2_gz_before_renamed" value="${['galatic', 'foxy']}"/> -->
   <xacro:include filename="$(find foxy_description)/urdf/base.xacro"/>
   <xacro:include filename="$(find foxy_description)/sensors/rgb_camera_generic.xacro"/>
@@ -23,9 +25,9 @@
     <origin xyz="0 0 0.12" rpy="0 0 0" />
   </xacro:lidar_generic>
-  <xacro:if value="${xacro.arg('system') == 'gz' and xacro.arg('distro') in ros2_gz_before_renamed}">
+  <xacro:if value="${xacro.arg('system') == 'sim' and xacro.arg('distro') in ros2_gz_before_renamed}">
     <!-- the plugin was renamed to gz_ros2_control from Iron -->
     <ros2_control name="GazeboSimSystem" type="system">
       <hardware>
-        <plugin>ign_ros2_control/IgnitionSystem</plugin>
+        <plugin>gz_ros2_control/GazeboSimSystem</plugin>
       </hardware>
       <joint name="left_wheel_joint">
@@ -48,8 +50,7 @@
     <gazebo>
       <!-- inserted at the top level of the <model> tag -->
-      <plugin filename="ignition-gazebo-sensors-system" name="ignition::gazebo::systems::Sensors">
-        <render_engine>ogre</render_engine>
+      <plugin filename="gz-sim-sensors-system" name="gz::sim::systems::Sensors">
       </plugin>
-      <plugin filename="ign_ros2_control-system" name="ign_ros2_control::IgnitionROS2ControlPlugin">
+      <plugin filename="gz_ros2_control-system" name="gz_ros2_control::GazeboSimROS2ControlPlugin">
         <ros>
           <namespace>${namespace}</namespace>
