Commit message: refactor sensor models and chasis

File: foxy_description/sensors/imu_generic.xacro (robot description, xacro)
@@ -1,28 +1,184 @@
 <?xml version="1.0"?>
 <robot xmlns:xacro="http://www.ros.org/wiki/xacro">
-  <xacro:macro name="imu_generic" params="name parent_link namespace system *origin">
+  <!-- MPU-6050 noise model. -->
+  <xacro:macro
+    name="mpu6050_axis_noise"
+    params="
+      stddev
+      bias_stddev
+      dynamic_bias_stddev
+      dynamic_bias_correlation_time
+      precision">
+    <noise type="gaussian_quantized">
+      <mean>0.0</mean>
+      <stddev>${stddev}</stddev>
+      <!-- Random constant bias selected when the simulation starts. -->
+      <bias_mean>0.0</bias_mean>
+      <bias_stddev>${bias_stddev}</bias_stddev>
+      <!-- Slowly changing bias / bias drift. -->
+      <dynamic_bias_stddev>
+        ${dynamic_bias_stddev}
+      </dynamic_bias_stddev>
+      <dynamic_bias_correlation_time>
+        ${dynamic_bias_correlation_time}
+      </dynamic_bias_correlation_time>
+      <!-- Approximate 16-bit ADC quantization. -->
+      <precision>${precision}</precision>
+    </noise>
+  </xacro:macro>
+  <!--
+    Gazebo approximation of an MPU-6050.
+    Default configuration:
+      gyro range:         +/-250 degrees/second
+      accelerometer:      +/-2 g
+      output rate:        100 Hz
+      orientation output: disabled
+    The MPU-6050 itself measures:
+      - three-axis angular velocity
+      - three-axis linear acceleration
+      - die temperature
+    It does not directly measure absolute orientation.
+  -->
+  <xacro:macro
+    name="imu_generic"
+    params="
+      name
+      parent_link
+      namespace
+      system
+      update_rate:=100.0
+      visualize:=false
+      enable_orientation:=false
+      gyro_noise_stddev:=0.000872665
+      gyro_bias_stddev:=0.00872665
+      gyro_dynamic_bias_stddev:=0.000174533
+      gyro_precision:=0.000133231
+      accel_noise_stddev:=0.02774
+      accel_bias_stddev:=0.0980665
+      accel_dynamic_bias_stddev:=0.00196133
+      accel_precision:=0.000598550
+      bias_correlation_time:=1000.0
+      *origin">
     <link name="${name}_link">
+      <!--
+        Approximate mass and inertia for a small MPU-6050 breakout board.
+        The link is fixed, so these values have negligible influence on the
+        robot dynamics.
+      -->
       <inertial>
-        <mass value="0.01"/>
-        <inertia ixx="0.000166667" ixy="0.0" ixz="0.0" iyy="0.000166667" iyz="0.0" izz="0.000166667"/>
+        <origin xyz="0 0 0" rpy="0 0 0"/>
+        <mass value="0.003"/>
+        <inertia
+          ixx="5.85e-8"
+          ixy="0.0"
+          ixz="0.0"
+          iyy="1.0225e-7"
+          iyz="0.0"
+          izz="1.5625e-7"/>
       </inertial>
+      <visual>
+        <geometry>
+          <box size="0.020 0.015 0.003"/>
+        </geometry>
+        <material name="${name}_pcb">
+          <color rgba="0.05 0.20 0.10 1.0"/>
+        </material>
+      </visual>
+      <collision>
+        <geometry>
+          <box size="0.020 0.015 0.003"/>
+        </geometry>
+      </collision>
     </link>
     <joint name="${name}_joint" type="fixed">
       <parent link="${parent_link}"/>
       <child link="${name}_link"/>
-      <xacro:insert_block name="origin" />
+      <xacro:insert_block name="origin"/>
     </joint>
+    <!-- Gazebo implementation exists only during simulation. -->
     <xacro:if value="${system == 'sim'}">
+      <!--
+        Required by Gazebo Sim for IMU sensor processing.
+        This should appear only once in the robot. The current Foxy
+        description contains one IMU, so keeping it here is acceptable.
+      -->
       <gazebo>
-        <plugin filename="gz-sim-imu-system"
-          name="gz::sim::systems::Imu">
-        </plugin>
+        <plugin
+          filename="gz-sim-imu-system"
+          name="gz::sim::systems::Imu"/>
       </gazebo>
       <gazebo reference="${name}_link">
         <sensor name="${name}" type="imu">
-          <always_on>1</always_on>
-          <update_rate>100</update_rate>
-          <visualize>true</visualize>
+          <pose>0 0 0 0 0 0</pose>
+          <always_on>true</always_on>
+          <update_rate>${update_rate}</update_rate>
+          <visualize>${visualize}</visualize>
           <topic>/${namespace}/${name}/imu</topic>
+          <!-- Gazebo Garden / Harmonic naming. -->
+          <gz_frame_id>${name}_link</gz_frame_id>
+          <!-- Compatibility with Gazebo Fortress-era sensor libraries. -->
+          <ignition_frame_id>${name}_link</ignition_frame_id>
+          <imu>
+            <!--
+              A raw MPU-6050 does not provide an absolute orientation
+              measurement. Orientation should be calculated by an external
+              filter or by software using the MPU DMP.
+            -->
+            <enable_orientation>${enable_orientation}</enable_orientation>
+            <!-- Gyroscope output, expressed in rad/s. -->
+            <angular_velocity>
+              <x>
+                <xacro:mpu6050_axis_noise
+                  stddev="${gyro_noise_stddev}"
+                  bias_stddev="${gyro_bias_stddev}"
+                  dynamic_bias_stddev="${gyro_dynamic_bias_stddev}"
+                  dynamic_bias_correlation_time="${bias_correlation_time}"
+                  precision="${gyro_precision}"/>
+              </x>
+              <y>
+                <xacro:mpu6050_axis_noise
+                  stddev="${gyro_noise_stddev}"
+                  bias_stddev="${gyro_bias_stddev}"
+                  dynamic_bias_stddev="${gyro_dynamic_bias_stddev}"
+                  dynamic_bias_correlation_time="${bias_correlation_time}"
+                  precision="${gyro_precision}"/>
+              </y>
+              <z>
+                <xacro:mpu6050_axis_noise
+                  stddev="${gyro_noise_stddev}"
+                  bias_stddev="${gyro_bias_stddev}"
+                  dynamic_bias_stddev="${gyro_dynamic_bias_stddev}"
+                  dynamic_bias_correlation_time="${bias_correlation_time}"
+                  precision="${gyro_precision}"/>
+              </z>
+            </angular_velocity>
+            <!-- Accelerometer output, expressed in m/s^2. -->
+            <linear_acceleration>
+              <x>
+                <xacro:mpu6050_axis_noise
+                  stddev="${accel_noise_stddev}"
+                  bias_stddev="${accel_bias_stddev}"
+                  dynamic_bias_stddev="${accel_dynamic_bias_stddev}"
+                  dynamic_bias_correlation_time="${bias_correlation_time}"
+                  precision="${accel_precision}"/>
+              </x>
+              <y>
+                <xacro:mpu6050_axis_noise
+                  stddev="${accel_noise_stddev}"
+                  bias_stddev="${accel_bias_stddev}"
+                  dynamic_bias_stddev="${accel_dynamic_bias_stddev}"
+                  dynamic_bias_correlation_time="${bias_correlation_time}"
+                  precision="${accel_precision}"/>
+              </y>
+              <z>
+                <xacro:mpu6050_axis_noise
+                  stddev="${accel_noise_stddev}"
+                  bias_stddev="${accel_bias_stddev}"
+                  dynamic_bias_stddev="${accel_dynamic_bias_stddev}"
+                  dynamic_bias_correlation_time="${bias_correlation_time}"
+                  precision="${accel_precision}"/>
+              </z>
+            </linear_acceleration>
+          </imu>
         </sensor>
       </gazebo>

File: foxy_description/sensors/rgb_camera_generic.xacro (robot description, xacro)
@@ -1,9 +1,74 @@
 <?xml version="1.0"?>
 <robot xmlns:xacro="http://www.ros.org/wiki/xacro">
-  <xacro:macro name="rgb_camera_generic" params="name parent_link namespace system *origin">
+  <!--
+    Waveshare RPi Camera (G) / OV5647 approximation.
+    Physical camera:
+      - OV5647, 5 MP
+      - 1920 x 1080 video mode
+      - 160 degree diagonal fisheye FoV
+      - 3.15 mm focal length
+      - manual focus
+      - rolling shutter
+    Simulation limitations:
+      - Gazebo does not model manual focus or rolling-shutter timing here.
+      - The fisheye projection is approximated with an equidistant lens.
+      - noise_stddev is a tunable simulation value, not a datasheet value.
+  -->
+  <xacro:macro
+    name="rgb_camera_generic"
+    params="
+      name
+      parent_link
+      namespace
+      system
+      image_width:=1920
+      image_height:=1080
+      update_rate:=30.0
+      horizontal_fov:=2.433898
+      near_clip:=0.05
+      far_clip:=100.0
+      noise_stddev:=0.007
+      visualize:=true
+      *origin">
+    <!--
+      Physical camera mounting frame.
+      ROS body-frame convention:
+        +X forward
+        +Y left
+        +Z up
+    -->
     <link name="${name}_link">
+      <visual>
+        <!--
+          Approximate envelope:
+            X: lens/module depth
+            Y: board width
+            Z: board height
+        -->
+        <origin xyz="-0.010 0 0" rpy="0 0 0"/>
+        <geometry>
+          <box size="0.010 0.015 0.014"/>
+        </geometry>
+        <material name="${name}_pcb_material">
+          <color rgba="0.05 0.15 0.05 1.0"/>
+        </material>
+      </visual>
+      <collision>
+        <origin xyz="-0.010 0 0" rpy="0 0 0"/>
+        <geometry>
+          <box size="0.020 0.025 0.024"/>
+        </geometry>
+      </collision>
+      <!-- Approximate 16 g mass including the camera assembly. -->
       <inertial>
-        <mass value="0.01"/>
-        <inertia ixx="0.000166667" ixy="0.0" ixz="0.0" iyy="0.000166667" iyz="0.0" izz="0.000166667"/>
+        <origin xyz="-0.010 0 0" rpy="0 0 0"/>
+        <mass value="0.016"/>
+        <inertia
+          ixx="1.6013e-6"
+          ixy="0.0"
+          ixz="0.0"
+          iyy="1.3013e-6"
+          iyz="0.0"
+          izz="1.3667e-6"/>
       </inertial>
     </link>
@@ -11,27 +76,75 @@
       <parent link="${parent_link}"/>
       <child link="${name}_link"/>
-      <xacro:insert_block name="origin" />
+      <xacro:insert_block name="origin"/>
     </joint>
+    <!--
+      REP-103 optical-frame convention:
+        +Z forward
+        +X right
+        +Y down
+    -->
+    <link name="${name}_optical_frame"/>
+    <joint name="${name}_optical_joint" type="fixed">
+      <parent link="${name}_link"/>
+      <child link="${name}_optical_frame"/>
+      <origin
+        xyz="0 0 0"
+        rpy="${-pi / 2} 0 ${-pi / 2}"/>
+    </joint>
+    <!-- Gazebo implementation exists only in simulation. -->
     <xacro:if value="${system == 'sim'}">
       <gazebo reference="${name}_link">
-        <plugin filename="gz-sim-imu-system"
-          name="gz::sim::systems::Imu">
-        </plugin>
-        <sensor name="${name}" type="camera">
-          <camera>
-            <horizontal_fov>1.047</horizontal_fov>
+        <!--
+          A normal camera uses a pinhole projection and is unsuitable for a
+          160-degree fisheye lens. Use Gazebo's wide-angle camera instead.
+        -->
+        <sensor name="${name}" type="wideanglecamera">
+          <pose>0 0 0 0 0 0</pose>
+          <always_on>true</always_on>
+          <update_rate>${update_rate}</update_rate>
+          <visualize>${visualize}</visualize>
+          <topic>/${namespace}/${name}/image</topic>
+          <frame_id>${name}_optical_frame</frame_id>
+          <camera name="${name}">
+            <camera_info_topic>
+              /${namespace}/${name}/camera_info
+            </camera_info_topic>
+            <!--
+              2.433898 rad = approximately 139.45 degrees horizontal.
+              With an equidistant projection and a 16:9 image, this
+              approximates the advertised 160-degree diagonal field of view.
+            -->
+            <horizontal_fov>${horizontal_fov}</horizontal_fov>
             <image>
-              <width>1080</width>
-              <height>720</height>
+              <width>${image_width}</width>
+              <height>${image_height}</height>
+              <format>R8G8B8</format>
+              <anti_aliasing>4</anti_aliasing>
             </image>
             <clip>
-              <near>0.1</near>
-              <far>100</far>
+              <near>${near_clip}</near>
+              <far>${far_clip}</far>
             </clip>
+            <!--
+              Equidistant is a reasonable generic fisheye approximation:
+                image radius is proportional to incident angle.
+              cutoff_angle is measured from the optical axis:
+                80 degrees = half of the advertised 160-degree diagonal FoV.
+            -->
+            <lens>
+              <type>equidistant</type>
+              <scale_to_hfov>true</scale_to_hfov>
+              <cutoff_angle>1.3962634</cutoff_angle>
+              <env_texture_size>1024</env_texture_size>
+            </lens>
+            <noise>
+              <type>gaussian</type>
+              <mean>0.0</mean>
+              <stddev>${noise_stddev}</stddev>
+            </noise>
+            <optical_frame_id>
+              ${name}_optical_frame
+            </optical_frame_id>
           </camera>
-          <always_on>1</always_on>
-          <update_rate>30</update_rate>
-          <visualize>true</visualize>
-          <topic>/${namespace}/${name}/image</topic>
         </sensor>
       </gazebo>

File: foxy_description/urdf/base.xacro (robot description, xacro)
@@ -5,21 +5,19 @@
   <xacro:property name="wheel_radius" value="0.033"/>
   <xacro:property name="wheel_width" value="0.025"/>
-  <xacro:property name="wheel_separation" value="0.101"/>
-  <xacro:property name="wheel_zoff" value="0.05"/>
-  <xacro:property name="wheel_xoff" value="0.04"/>
-  <xacro:property name="caster_radius" value="0.009"/>
-  <xacro:property name="caster_zoff" value="0.032"/>
-  <xacro:property name="caster_xoff" value="-0.043"/>
+  <xacro:property name="wheel_separation" value="0.1045"/>
+  <xacro:property name="wheel_zoff" value="0.01235"/>
+  <xacro:property name="wheel_xoff" value="0.025"/>
+  <xacro:property name="caster_radius" value="0.01"/>
+  <xacro:property name="caster_zoff" value="0.035"/>
+  <xacro:property name="caster_xoff" value="-0.0585"/>
   <xacro:include filename="$(find foxy_description)/urdf/utils.xacro"/>
-  <xacro:macro name="wheel" params="prefix parent x_reflect y_reflect">
+  <xacro:macro name="wheel" params="prefix parent reflect">
     <link name="${prefix}_link">
       <visual>
-        <origin xyz="0 0 0" rpy="${pi/2} 0 0"/>
+        <!-- reflect =  1 -> +180 degrees around Z reflect = -1 -> -180 degrees around Z -->
+        <origin xyz="0 0 0" rpy="0 0 ${(1 - reflect) * pi / 2}"/>
         <geometry>
-          <cylinder radius="${wheel_radius}" length="${wheel_width}"/>
+          <mesh filename="model://foxy_description/meshes/wheel.obj"/>
         </geometry>
-        <material name="Gray">
-          <color rgba="0.5 0.5 0.5 1.0"/>
-        </material>
       </visual>
       <collision>
@@ -34,5 +32,9 @@
       <parent link="${parent}"/>
       <child link="${prefix}_link"/>
-      <origin xyz="${x_reflect*wheel_xoff} ${y_reflect*(wheel_separation/2)} ${-wheel_zoff}" rpy="0 0 0"/>
+      <origin
+      xyz="${wheel_xoff}
+           ${reflect * (wheel_separation / 2)}
+           ${-wheel_zoff}"
+      rpy="0 0 0"/>
       <axis xyz="0 1 0"/>
     </joint>
@@ -56,14 +58,13 @@
       <visual>
         <geometry>
-          <box size="${base_length} ${base_width} ${base_height}"/>
+          <mesh filename="model://foxy_description/meshes/foxy-chasis.obj"/>
+          <!-- <box size="${base_length} ${base_width} ${base_height}"/> -->
         </geometry>
-        <geometry>
-          <box size="0.6 0.4 0.2" />
-        </geometry>
-        <material name="green" />
       </visual>
       <collision>
+        <origin xyz="0 0 0.03" rpy="0 0 0"/>
         <geometry>
-          <box size="${base_length} ${base_width} ${base_height}"/>
+          <!-- <box size="${base_length} ${base_width} ${base_height}"/> -->
+          <box size="0.21 0.06 0.128"/>
         </geometry>
       </collision>
@@ -75,6 +76,6 @@
       <dynamics friction="1.0"/>
     </joint>
-    <xacro:wheel prefix="left_wheel" parent="${root_frame}" x_reflect="1" y_reflect="1" />
-    <xacro:wheel prefix="right_wheel" parent="${root_frame}" x_reflect="1" y_reflect="-1" />
+    <xacro:wheel prefix="left_wheel" parent="${root_frame}" reflect="1" />
+    <xacro:wheel prefix="right_wheel" parent="${root_frame}" reflect="-1" />
     <link name="caster_wheel">
       <visual>
@@ -94,5 +95,5 @@
       <parent link="${root_frame}" />
       <child link="caster_wheel" />
-      <origin xyz="${caster_xoff} 0 -${(wheel_radius+wheel_zoff)-caster_radius}" rpy="0 0 0" />
+      <origin xyz="${caster_xoff} 0 -${caster_zoff}" rpy="0 0 0" />
     </joint>
   </xacro:macro>

File: foxy_description/urdf/foxy.urdf.xacro (robot description, xacro)
@@ -15,14 +15,18 @@
   <xacro:include filename="$(find foxy_description)/sensors/imu_generic.xacro"/>
   <xacro:include filename="$(find foxy_description)/sensors/lidar_generic.xacro"/>
+  <xacro:include filename="$(find foxy_description)/sensors/vl53l0x.xacro"/>
   <xacro:foxy_base root_frame="${root_frame}"/>
   <xacro:rgb_camera_generic name="front_camera" parent_link="${root_frame}" namespace="${namespace}" system="${xacro.arg('system')}">
-    <origin xyz="0.075 0 0.07" rpy="0.0 0.13 0" />
+    <origin xyz="0.08938 0 0.07209" rpy="0.0 ${radians(16.1)} 0" />
   </xacro:rgb_camera_generic>
   <xacro:imu_generic name="imu_sensor" parent_link="${root_frame}" namespace="${namespace}" system="${xacro.arg('system')}">
     <origin xyz="0 0 0" rpy="0 0 0" />
   </xacro:imu_generic>
-  <xacro:lidar_generic name="lidar_sensor" parent_link="${root_frame}" namespace="${namespace}" system="${xacro.arg('system')}">
-    <origin xyz="0 0 0.12" rpy="0 0 0" />
-  </xacro:lidar_generic>
+  <xacro:vl53l0x name="vl53l0x/front" parent_link="${root_frame}" namespace="${namespace}" system="${xacro.arg('system')}" visualize="true">
+    <origin xyz="0.10678 0 0.037" rpy="0 0 0" />
+  </xacro:vl53l0x>
+  <!-- <xacro:lidar_generic name="lidar_sensor" parent_link="${root_frame}" namespace="${namespace}" system="${xacro.arg('system')}"> -->
+  <!--   <origin xyz="0 0 0.12" rpy="0 0 0" /> -->
+  <!-- </xacro:lidar_generic> -->
   <xacro:if value="${xacro.arg('system') == 'sim' and xacro.arg('distro') in ros2_gz_before_renamed}">
     <!-- the plugin was renamed to gz_ros2_control from Iron -->
